File: piezamp.kicad_pcb (KiCad board)
At the start: 2 copper layers, 64.1 x 41.4 mm, 54 parts, among them J3 Output (TRS), J4 Power_Conn, J5 Piezo A, J6 Piezo B, SW1 Power, SW2 Mode / Polarity, U1 NE5532DR, U2 NE5532DR

Commit message: More vias, highlight the ground pin
Parts:
- removed the J4 at (102.5, 129.2)
- removed J5: Piezo A, Connector_PinHeader_2.54mm:PinHeader_1x02_P2.54mm_Vertical
- removed J6: Piezo B, Connector_PinHeader_2.54mm:PinHeader_1x02_P2.54mm_Vertical
- removed R25, R26, R27: 10k, Resistor_SMD:R_0603_1608Metric
- added J1: Piezo A, Connector_PinHeader_2.54mm:PinHeader_1x02_P2.54mm_Vertical, F.Cu at (102.6, 105.2)
- added J2: Piezo B, Connector_PinHeader_2.54mm:PinHeader_1x02_P2.54mm_Vertical, F.Cu at (102.6, 119.6)
- added J3: Power_Conn, Connector_PinHeader_2.54mm:PinHeader_1x02_P2.54mm_Vertical, F.Cu at (102.6, 131.8)
- added R15: 10k, Resistor_SMD:R_0603_1608Metric, F.Cu at (138.2, 114.3)
- added R16: 10k, Resistor_SMD:R_0603_1608Metric, F.Cu at (140.0, 116.6)
- added R17: 10k, Resistor_SMD:R_0603_1608Metric, F.Cu at (138.2, 117.8)
- moved U2 0.09 mm to (145.0, 114.0)
- moved SW1 0.08 mm to (102.6, 136.8)
- renumbered RV3 to BLEND1, C10 to C1, C33 to C10, C34 to C11, C31 to C12, C40 to C13, C42 to C14, C32 to C15, C41 to C16, C20 to C2, C11 to C3, C21 to C4, C30 to C5, C12 to C6, C22 to C7, C13 to C8, C23 to C9, D10 to D1, D11 to D2, D20 to D3, D21 to D4, D1 to D5, RV1 to GAIN_A1, RV2 to GAIN_B1, J3 to J4, RV4 to LPF1, RV5 to MASTER_VOL1, R10 to R1, R31 to R10, R32 to R11, R14 to R12, R24 to R13, R33 to R14, R42 to R18, R40 to R19, R20 to R2, R41 to R20, R11 to R3, R21 to R4, R12 to R5, R22 to R6, R30 to R7, R13 to R8, R23 to R9
Routing:
- net Net-(J2-Pin_2): track 4.66 -> 7.44 mm
- net GND: vias 7 -> 27
- net (no net): vias 0 -> 2
Other:
- board text added: "GND >"
