File: piezamp.kicad_sch (KiCad schematic)
At the start: 54 parts, among them J3 Output (TRS), J4 Power_Conn, J5 Piezo A, J6 Piezo B, SW1 Power, SW2 Mode / Polarity, U1 NE5532DR, U2 NE5532DR

Commit message: Update README and schem
Other:
- company: Peek Robotics -> GOBLINOMIX HEAVY INDUSTRIES
- title: Dual Piezo Preamp (NE5532) -> PiezAmp
Changed lines of the file:
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@@
 	(paper "A3")
 	(title_block
-		(title "Dual Piezo Preamp (NE5532)")
+		(title "PiezAmp")
 		(date "2026-09-25")
-		(rev "0.1")
-		(company "Peek Robotics")
-		(comment 1 "Copyright 2026")
-		(comment 2 "Designed by: Laurence")
-		(comment 3 "See PLAN.md for design rationale")
+		(rev "1.0")
+		(company "GOBLINOMIX HEAVY INDUSTRIES")
+		(comment 1 "Based off Richard Mudhar's design")
+		(comment 2 "https://www.richardmudhar.com/blog/piezo-contact-microphone-hi-z-amplifier-low-noise-version/")
+	)
+	(rectangle
+		(start 13.97 36.83)
+		(end 128.27 95.25)
+		(stroke
+			(width 0)
+			(type default)
+		)
+		(fill
+			(type none)
+		)
+	)
+	(rectangle
+		(start 186.69 77.47)
+		(end 294.64 120.65)
+		(stroke
+			(width 0)
+			(type default)
+		)
+		(fill
+			(type none)
+		)
+	)
+	(rectangle
+		(start 13.97 96.52)
+		(end 127 171.45)
+		(stroke
+			(width 0)
+			(type default)
+		)
+		(fill
+			(type none)
+		)
+	)
+	(rectangle
+		(start 128.27 111.76)
+		(end 198.12 153.67)
+		(stroke
+			(width 0)
+			(type default)
+		)
+		(fill
+			(type none)
+		)
 	)
 	(text "High-cut (LPF) fc = 1 / (2 pi (RV4 + blend source) C40) = 27 kHz...34 Hz, CW = more cut\nR40 isolates C40 from A_OUT in stereo mode"

Commit message: did some renders, annotated schematic
Parts:
- renumbered RV3 to BLEND, RV1 to GAIN_A, RV2 to GAIN_B, RV4 to LPF, RV5 to MASTER_VOL
Other:
- note added: "An extra inverting opamp stage flips the signal from preamp B when engaged (SW2-1 turns it on / off)"
- note added: "BLEND -> LPF -> BUFFER -> MASTER VOL"
- note added: "Low pass filter fc = 1 / (2 pi (RV4 + blend source) C40) = 27 kHz...34 Hz If you want to wire the filter as a pot you intend to control, find an log taper one because the linear ones will have a really small usable range (fine for trim) Volume pot works okay as linear, but log is better!"
- note added: "OP-AMP SUPPLIES"
- note added: "PHASE INVERT"
- note added: "POWER"
- note added: "PREAMP A (gain = 1 + (R13+GAIN_A)/R12 = x2...x12, CW = more gain)"
- note added: "PREAMP B (identical to A)"
- note added: "The voltage divider here provides a halfway point for VREF So say if you have 9v in, VREF is the midpoint at 4.5v and the audio signal from the opamps is centered around there"
- note added: "There's some fuckery here so that it can be wired for mono, or for stereo (Stero bypasses everything after and including the blend) MONO blend -> low-cut -> volume -> tip (TS or TRS lead): 2 OFF, 3 OFF, 4 OFF STEREO A -> tip, B -> ring, no blend/filter/volume (TRS lead): 2 ON, 3 ON, 4 ON 1 = B polarity 2 = A direct 3 = volume bypass 4 = B to ring"
- note removed: "BLEND (RV3) -> HIGH-CUT LPF (RV4) -> BUFFER -> MASTER (RV5)"
- note removed: "High-cut (LPF) fc = 1 / (2 pi (RV4 + blend source) C40) = 27 kHz...34 Hz, CW = more cut R40 isolates C40 from A_OUT in stereo mode"
- note removed: "MONO blend -> low-cut -> volume -> tip (TS or TRS lead): 2 OFF, 3 OFF, 4 OFF STEREO A -> tip, B -> ring, no blend/filter/volume (TRS lead): 2 ON, 3 ON, 4 ON 1 = B polarity 2 = A direct 3 = volume bypass 4 = B to ring"
- note removed: "OP-AMP SUPPLIES (C31/C32 at pin 8)"
- note removed: "POLARITY B (SW2-1 off = +1, on = -1)"
- note removed: "POWER (9-18 V DC via J4; DC jack, battery and switch wired off-board)"
- note removed: "PREAMP A (gain = 1 + (R13+RV1)/R12 = x2...x12, CW = more gain)"
- note removed: "PREAMP B (identical to A, gain trim RV2)"
- note removed: "VREF = V+/2 for the signal stages; VREF_IN is a separately filtered copy for the 1M input bias only - do not merge"
- moved on the sheet: BLEND, C10, C11, C12, C13, C30, C31, C32, C33, C34, C40, C41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

Commit message: More vias, highlight the ground pin
Parts:
- removed J4: Power_Conn, Connector_PinHeader_2.54mm:PinHeader_1x02_P2.54mm_Vertical, symbol Connector_Generic:Conn_01x02
- removed J5: Piezo A, Connector_PinHeader_2.54mm:PinHeader_1x02_P2.54mm_Vertical, symbol Connector_Generic:Conn_01x02
- removed J6: Piezo B, Connector_PinHeader_2.54mm:PinHeader_1x02_P2.54mm_Vertical, symbol Connector_Generic:Conn_01x02
- added J1: Piezo A, Connector_PinHeader_2.54mm:PinHeader_1x02_P2.54mm_Vertical, symbol Connector_Generic:Conn_01x02
- added J2: Piezo B, Connector_PinHeader_2.54mm:PinHeader_1x02_P2.54mm_Vertical, symbol Connector_Generic:Conn_01x02
- added J3: Power_Conn, Connector_PinHeader_2.54mm:PinHeader_1x02_P2.54mm_Vertical, symbol Connector_Generic:Conn_01x02
- renumbered BLEND to BLEND1, C10 to C1, C33 to C10, C34 to C11, C31 to C12, C40 to C13, C42 to C14, C32 to C15, C41 to C16, C20 to C2, C11 to C3, C21 to C4, C30 to C5, C12 to C6, C22 to C7, C13 to C8, C23 to C9, D10 to D1, D11 to D2, D20 to D3, D21 to D4, D1 to D5, GAIN_A to GAIN_A1, GAIN_B to GAIN_B1, J3 to J4, LPF to LPF1, MASTER_VOL to MASTER_VOL1, R10 to R1, R31 to R10, R32 to R11, R14 to R12, R24 to R13, R33 to R14, R25 to R15, R27 to R16, R26 to R17, R42 to R18, R40 to R19, R20 to R2, R41 to R20, R11 to R3, R21 to R4, R12 to R5, R22 to R6, R30 to R7, R13 to R8, R23 to R9
Connections:
- net GND: now also J1.1 (Pin_1), J2.1 (Pin_1), J3.1 (Pin_1)
- net at SW1.1 (A): now also J3.2 (Pin_2)
- net at C1.1: now also J1.2 (Pin_2)
- net at C2.1: now also J2.2 (Pin_2)
